Commit message: working tf visualisation

File: rotors_description/urdf/component_snippets.xacro (robot description, xacro)
@@ -71,4 +71,5 @@
     </joint>
     <gazebo reference="${namespace}/camera_${camera_suffix}_link">
+      <material>Gazebo/Black</material>
       <sensor type="camera" name="${namespace}_camera_${camera_suffix}">
         <update_rate>${frame_rate}</update_rate>
